File: Arduino/REV11/rev11.brd (EAGLE design)
At the start: 79 x 79 mm, 28 parts, among them IC2 ATMEGA168-AU, Q1 32768Hz, U1 TC1185SMD

Commit message: update rev11
Parts:
- removed C1, C2: 10uF 10V, resistor:C0603
- removed U1: TC1185SMD, 3.3VREG:TC1185
- removed X1: (no value), con-wago-500:W237-102
- added +, -: (no value), wirepad:2,15/1,0
- moved R2 61.5 mm to (17.8, 47.6), turned to 270 degrees
- moved R10 12.3 mm to (73.1, 29.0), turned to 90 degrees
- moved R5 5.54 mm to (68.7, 15.0), turned to 270 degrees
- moved C11 5.34 mm to (63.3, 15.1)
- moved R12 2.54 mm to (15.2, 47.6)
- moved R4 1.66 mm to (66.1, 15.1), turned to 270 degrees
- moved ANT 1.27 mm to (24.8, 76.8)
- moved LED 1.27 mm to (2.05, 52.5)
- moved RFM23B 1.00 mm to (70.1, 40.5)
Connections:
- removed net 5V: C1.1, FTDI+I2C.12, U1.1, U1.3
- net BOILER: no longer FTDI+I2C.6
- net GND: now also -.1; no longer C1.2, C2.1, U1.2, X1.2
- net VCC: now also +.1; no longer C2.2, U1.5
Other:
- board text removed: "3.3"
- board text removed: "5"
- board text removed: "B"
