File: Arduino/REV11/rev11.sch (EAGLE design)
At the start: 24 parts, among them IC2 ATMEGA168-AU, Q1 32768Hz

Commit message: update rev11
Other:
- note removed: "2"
- note removed: "Author(s) / Copyright (s): Bo Herrmannsen 2013--2014, Damon Hart-Davis 2013--2014, Mike Stirling 2013"
- note removed: "OpenTRV Wireless TRV Controller"
Changed lines of the file:
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@@
 <text x="7.62" y="15.24" size="1.778" layer="91">software, hardware and materials distributed under this Licence</text>
 <text x="7.62" y="12.7" size="1.778" layer="91">is distributed on an "AS IS" BASIS, WITHOUT WARRANTIES OR CONDITIONS</text>
-<text x="7.62" y="2.54" size="1.778" layer="91">Author(s) / Copyright (s): Bo Herrmannsen 2013--2014, Damon Hart-Davis 2013--2014, Mike Stirling 2013</text>
-<text x="289.56" y="33.02" size="1.778" layer="91">OpenTRV Wireless TRV Controller</text>
 <text x="7.62" y="10.16" size="1.778" layer="91"></text>
 <text x="7.62" y="10.16" size="1.778" layer="91">OF ANY KIND, either express or implied. See the Licence for the</text>
@@
 <wire x1="93.98" y1="160.02" x2="157.48" y2="160.02" width="0.3048" layer="94"/>
 <wire x1="93.98" y1="264.16" x2="93.98" y2="208.28" width="0.3048" layer="94"/>
-<text x="378.46" y="10.16" size="1.778" layer="91">2</text>
 <wire x1="157.48" y1="208.28" x2="157.48" y2="160.02" width="0.3048" layer="94"/>
 <text x="350.52" y="251.46" size="1.778" layer="91">50 ohm track 86mm</text>

Commit message: update rev11
Connections:
- net BOILER renamed D6
- net LED_HEATCALL_L renamed LED
- net N$11 renamed A1
- net N$14 renamed A0
- net N$16 renamed A2
- net N$19 renamed D8
- net N$20 renamed D5
- net N$21 renamed D7
- net N$22 renamed D2
- net N$30 renamed D3
- new net A3: IC2.ANALOG_3
- new net A6: IC2.ANALOG_6
- new net A7: IC2.ANALOG_7
Changed lines of the file:
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@@
 </segment>
 </net>
-<net name="BOILER" class="0">
+<net name="D6" class="0">
 <segment>
 <wire x1="228.6" y1="81.28" x2="248.92" y2="81.28" width="0.1524" layer="91"/>
 <pinref part="IC2" gate="1" pin="DIGITAL_6(PWM)"/>
+<label x="251.46" y="81.28" size="1.778" layer="95"/>
 </segment>
 </net>
@@
 </segment>
 </net>
-<net name="LED_HEATCALL_L" class="0">
-<segment>
-<pinref part="R7" gate="G$1" pin="1"/>
-<wire x1="68.58" y1="220.98" x2="68.58" y2="226.06" width="0.1524" layer="91"/>
-<label x="60.96" y="220.98" size="1.778" layer="95"/>
-</segment>
-<segment>
-<wire x1="228.6" y1="86.36" x2="248.92" y2="86.36" width="0.1524" layer="91"/>
-<label x="251.46" y="86.36" size="1.778" layer="95"/>
-<pinref part="IC2" gate="1" pin="DIGITAL_4"/>
-</segment>
-</net>
 <net name="RESET" class="0">
 <segment>
@@
 </segment>
 </net>
-<net name="N$14" class="0">
+<net name="A0" class="0">
 <segment>
 <wire x1="248.92" y1="119.38" x2="228.6" y2="119.38" width="0.1524" layer="91"/>
 <pinref part="IC2" gate="1" pin="ANALOG_0"/>
-</segment>
-</net>
-<net name="N$16" class="0">
+<label x="251.46" y="119.38" size="1.778" layer="95"/>
+</segment>
+</net>
+<net name="A2" class="0">
 <segment>
 <wire x1="248.92" y1="114.3" x2="228.6" y2="114.3" width="0.1524" layer="91"/>
 <pinref part="IC2" gate="1" pin="ANALOG_2"/>
-</segment>
-</net>
-<net name="N$20" class="0">
+<label x="251.46" y="114.3" size="1.778" layer="95"/>
+</segment>
+</net>
+<net name="D5" class="0">
 <segment>
 <wire x1="228.6" y1="83.82" x2="248.92" y2="83.82" width="0.1524" layer="91"/>
 <pinref part="IC2" gate="1" pin="DIGITAL_5(PWM)"/>
-</segment>
-</net>
-<net name="N$21" class="0">
+<label x="251.46" y="83.82" size="1.778" layer="95"/>
+</segment>
+</net>
+<net name="D7" class="0">
 <segment>
 <wire x1="228.6" y1="78.74" x2="248.92" y2="78.74" width="0.1524" layer="91"/>
 <pinref part="IC2" gate="1" pin="DIGITAL_7"/>
-</segment>
-</net>
-<net name="N$19" class="0">
+<label x="251.46" y="78.74" size="1.778" layer="95"/>
+</segment>
+</net>
+<net name="D8" class="0">
 <segment>
 <wire x1="228.6" y1="73.66" x2="248.92" y2="73.66" width="0.1524" layer="91"/>
 <pinref part="IC2" gate="1" pin="DIGITAL_8"/>
-</segment>
-</net>
-<net name="N$22" class="0">
+<label x="251.46" y="73.66" size="1.778" layer="95"/>
+</segment>
+</net>
+<net name="D2" class="0">
 <segment>
 <wire x1="248.92" y1="91.44" x2="228.6" y2="91.44" width="0.1524" layer="91"/>
 <pinref part="IC2" gate="1" pin="DIGITAL_2"/>
-</segment>
-</net>
-<net name="N$11" class="0">
+<label x="251.46" y="91.44" size="1.778" layer="95"/>
+</segment>
+</net>
+<net name="A1" class="0">
 <segment>
 <pinref part="IC2" gate="1" pin="ANALOG_1"/>
 <wire x1="228.6" y1="116.84" x2="248.92" y2="116.84" width="0.1524" layer="91"/>
-</segment>
-</net>
-<net name="N$30" class="0">
+<label x="251.46" y="116.84" size="1.778" layer="95"/>
+</segment>
+</net>
+<net name="D3" class="0">
 <segment>
 <pinref part="IC2" gate="1" pin="DIGITAL_3(PWM)"/>
 <wire x1="228.6" y1="88.9" x2="248.92" y2="88.9" width="0.1524" layer="91"/>
-</segment>
-</net>
+<label x="251.46" y="88.9" size="1.778" layer="95"/>
+</segment>
+</net>
+<net name="A3" class="0">
+<segment>
+<pinref part="IC2" gate="1" pin="ANALOG_3"/>
+<wire x1="228.6" y1="111.76" x2="248.92" y2="111.76" width="0.1524" layer="91"/>
+<label x="251.46" y="111.76" size="1.778" layer="95"/>
+</segment>
+</net>
+<net name="A6" class="0">
+<segment>
+<pinref part="IC2" gate="1" pin="ANALOG_6"/>
+<wire x1="228.6" y1="104.14" x2="248.92" y2="104.14" width="0.1524" layer="91"/>
+<label x="251.46" y="104.14" size="1.778" layer="95"/>
+</segment>
+</net>
+<net name="A7" class="0">
+<segment>
+<pinref part="IC2" gate="1" pin="ANALOG_7"/>
+<wire x1="228.6" y1="101.6" x2="248.92" y2="101.6" width="0.1524" layer="91"/>
+<label x="251.46" y="101.6" size="1.778" layer="95"/>
+</segment>
+</net>
+<net name="LED" class="0">
+<segment>
+<wire x1="228.6" y1="86.36" x2="248.92" y2="86.36" width="0.1524" layer="91"/>
+<label x="251.46" y="86.36" size="1.778" layer="95"/>
+<pinref part="IC2" gate="1" pin="DIGITAL_4"/>
+</segment>
+<segment>
+<pinref part="R7" gate="G$1" pin="1"/>
+<wire x1="68.58" y1="220.98" x2="68.58" y2="226.06" width="0.1524" layer="91"/>
+<label x="66.04" y="218.44" size="1.778" layer="95"/>
+</segment>
+</net>
