File: Arduino/hardware/REV10/rev10.brd (EAGLE design)
At the start: 100 x 80 mm, 48 parts, among them IC2 ATMEGA168-AU, Q1 32768Hz, U1 TC1185SMD, U2 ARDUINO

Commit message: almost routed rev10, one wire left
just in case my pc blows up
Parts:
- moved R3 44.1 mm to (83.8, 40.6), turned to 90 degrees
- moved C5 39.8 mm to (80.4, 35.6)
- moved R1 39.4 mm to (80.0, 41.9), turned to 90 degrees
- moved C12 20.8 mm to (65.6, 27.4), turned to 270 degrees
- moved R17 19.7 mm to (73.0, 28.6), turned to 90 degrees
- moved C9 17.5 mm to (80.6, 55.7), turned to 90 degrees
- moved R9 12.0 mm to (75.9, 41.3), turned to 90 degrees
- moved R6 10.8 mm to (67.9, 5.08), turned to 90 degrees
- moved R15 9.46 mm to (76.7, 33.7), turned to 90 degrees
- moved R16 9.15 mm to (53.3, 39.6)
- moved IC2 8.89 mm to (66.0, 36.8)
- moved PFET 8.89 mm to (81.9, 27.3)
- moved Q1 8.89 mm to (63.9, 49.7)
- moved R10 8.89 mm to (71.0, 56.7)
- moved R12 8.89 mm to (66.0, 57.8)
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Routing:
- net VCC: track 4.73 -> 254.4 mm
- net 5V: track 0.00 -> 184.1 mm, vias 0 -> 3
- net D2: track 0.09 -> 151.8 mm, vias 0 -> 1
- net N$5: track 0.00 -> 130.5 mm, vias 0 -> 1
- net SCL: track 4.58 -> 132.4 mm, vias 0 -> 3
- net SDA: track 4.58 -> 131.5 mm, vias 0 -> 4
- net N$30: track 0.00 -> 117.5 mm, vias 0 -> 1
- net SPI_NSS: track 0.00 -> 116.9 mm, vias 0 -> 2
- net SPI_SCK: track 0.00 -> 99.1 mm, vias 0 -> 4
- net VOICE: track 0.00 -> 97.8 mm, vias 0 -> 2
- net N$26: track 0.00 -> 96.8 mm, vias 0 -> 3
- net SPI_MOSI: track 0.00 -> 93.7 mm, vias 0 -> 4
- net N$28: track 0.00 -> 87.9 mm, vias 0 -> 4
- net N$25: track 0.00 -> 82.3 mm, vias 0 -> 4
- net SPI_MISO: track 0.00 -> 82.1 mm, vias 0 -> 3
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
Commit message: rev10 all routed :-D
Parts:
- moved C12 1.12 mm to (65.6, 28.5)
Routing:
- net N$6: track 4.48 -> 3.27 mm
- net GND: vias 30 -> 31
Changed lines of the file:
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@@
 </element>
 <element name="U$1" library="ohw-logo" package="OSHW_10X200_NOTEXT" value="" x="14.674165625" y="32.53610625"/>
-<element name="C12" library="resistor" package="C0603" value="100nF" x="65.64" y="27.3806125" smashed="yes" rot="R270">
-<attribute name="NAME" x="64.388" y="26.3003875" size="1" layer="25" font="vector" rot="R90"/>
+<element name="C12" library="resistor" package="C0603" value="100nF" x="65.64" y="28.5" smashed="yes" rot="R270">
+<attribute name="NAME" x="64.388" y="27.419775" size="1" layer="25" font="vector" rot="R90"/>
 </element>
 <element name="R10" library="resistor" package="R0603" value="1K" x="71.0096125" y="56.7020875" smashed="yes" rot="R90">
@@
 <via x="40.64" y="28.575" extent="1-16" drill="0.5"/>
 <via x="64.77" y="23.495" extent="1-16" drill="0.5"/>
-<wire x1="65.64" y1="41.1226" x2="65.93" y2="45.58" width="0" layer="19" extent="1-1"/>
+<via x="62.12" y="67.31" extent="1-16" drill="0.5"/>
 </signal>
 <signal name="SPI_SCK">
@@
 <contactref element="C12" pad="1"/>
 <contactref element="IC2" pad="20"/>
-<wire x1="65.75" y1="32.5" x2="65.75" y2="28.25" width="0.4064" layer="1"/>
-<wire x1="65.75" y1="28.25" x2="65.64" y2="28.2306125" width="0.4064" layer="1"/>
+<wire x1="65.75" y1="32.5" x2="65.75" y2="30.79" width="0.4064" layer="1"/>
+<wire x1="65.75" y1="30.79" x2="65.64" y2="29.35" width="0.4064" layer="1"/>
 <wire x1="65.75" y1="32.5" x2="65.64" y2="32.5374" width="0.4064" layer="1"/>
 </signal>
