File: Arduino/hardware/REV10/rev10.sch (EAGLE design)
At the start: 46 parts, among them IC2 ATMEGA168-AU, Q1 32768Hz, U1 TC1185SMD, U2 ARDUINO

Commit message: rev 10 with 5 tracks left
Parts:
- removed C5: 100nF, resistor:C-EUC0603
Connections:
- removed net N$25: C5.2, I2C_EXT.5
- net RESET: now also I2C_EXT.5; no longer C5.1
Changed lines of the file:
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@@
 <part name="R1" library="resistor" deviceset="R-EU_" device="R0603" value="4.7K"/>
 <part name="R3" library="resistor" deviceset="R-EU_" device="R0603" value="4.7K"/>
-<part name="C5" library="resistor" deviceset="C-EU" device="C0603" value="100nF"/>
 <part name="I2C_EXT" library="pinhead" deviceset="PINHD-2X7" device=""/>
 <part name="IC2" library="Arduino-AVR" deviceset="ATMEGA168" device="-AU"/>
@@
 <text x="17.78" y="139.7" size="1.778" layer="94">On BOM</text>
 <text x="134.62" y="195.58" size="1.778" layer="94" rot="R90">On BOM</text>
-<text x="124.46" y="203.2" size="1.778" layer="94" rot="R180">On BOM</text>
 <text x="129.54" y="226.06" size="1.778" layer="94">On BOM</text>
 <text x="205.74" y="231.14" size="1.778" layer="94" rot="R90">On BOM</text>
@@
 <instance part="R1" gate="G$1" x="129.54" y="200.66" rot="R90"/>
 <instance part="R3" gate="G$1" x="129.54" y="226.06" rot="R270"/>
-<instance part="C5" gate="G$1" x="121.92" y="200.66" rot="R180"/>
 <instance part="I2C_EXT" gate="A" x="124.46" y="213.36" rot="R90"/>
 <instance part="IC2" gate="1" x="195.58" y="91.44"/>
@@
 </segment>
 <segment>
-<pinref part="C5" gate="G$1" pin="1"/>
-<wire x1="121.92" y1="198.12" x2="121.92" y2="190.5" width="0.1524" layer="91"/>
 <label x="121.92" y="187.96" size="1.778" layer="95" rot="R270"/>
+<pinref part="I2C_EXT" gate="A" pin="5"/>
+<wire x1="121.92" y1="190.5" x2="121.92" y2="210.82" width="0.1524" layer="91"/>
 </segment>
 <segment>
@@
 </segment>
 </net>
-<net name="N$25" class="0">
-<segment>
-<wire x1="121.92" y1="210.82" x2="121.92" y2="205.74" width="0.1524" layer="91"/>
-<pinref part="C5" gate="G$1" pin="2"/>
-<pinref part="I2C_EXT" gate="A" pin="5"/>
-</segment>
-</net>

Commit message: latest work for rev10
Parts:
- removed JP2: (no value), pinhead:PINHD-2X3
- added C5: 100nF, resistor:C-EUC0603
- added JP1: (no value), pinhead:PINHD-2X3
- I2C_EXT: device pinhead:PINHD-2X7 -> pinhead:PINHD-2X10
Connections:
- removed net N$28: I2C_EXT.11, R1.2
- new net N$24: I2C_EXT.18, R1.2
- new net N$25: I2C_EXT.16, R3.2
- net 5V: now also JP1.2; no longer JP2.4
- net D2: now also I2C_EXT.17; no longer I2C_EXT.14
- net GND: now also I2C_EXT.10, I2C_EXT.12, JP1.6; no longer JP2.5
- net IO_POWER_UP: now also I2C_EXT.19
- net N$1: now also JP1.4; no longer JP2.1
- net N$26: now also C5.2, I2C_EXT.5; no longer I2C_EXT.12, R3.2
- net N$5: now also JP1.3; no longer JP2.3
- net RESET: now also C5.1; no longer I2C_EXT.5
- net RFM_IRQ: now also I2C_EXT.13; no longer I2C_EXT.7
- net SDA: now also I2C_EXT.11; no longer I2C_EXT.10
- net SPI_NSS: now also I2C_EXT.15; no longer I2C_EXT.8
- net VCC: now also JP1.1; no longer JP2.6
- net VOICE: now also JP1.5; no longer JP2.2
Other:
- moved on the sheet: DQ, R1, R3

Commit message: minor changes to rev10
Changed lines of the file:
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@@
 <wire x1="93.98" y1="91.44" x2="0" y2="91.44" width="0.3048" layer="94"/>
 <wire x1="93.98" y1="160.02" x2="93.98" y2="91.44" width="0.3048" layer="94"/>
-<text x="327.66" y="160.02" size="1.778" layer="94">On BOM</text>
-<text x="327.66" y="185.42" size="1.778" layer="94">On BOM</text>
-<text x="231.14" y="213.36" size="1.778" layer="94">On BOM</text>
-<text x="60.96" y="243.84" size="1.778" layer="94">On BOM</text>
-<text x="22.86" y="119.38" size="1.778" layer="94">On BOM</text>
-<text x="162.56" y="210.82" size="1.778" layer="94">On BOM</text>
+<text x="345.44" y="167.64" size="1.778" layer="94">On BOM</text>
+<text x="350.52" y="193.04" size="1.778" layer="94">On BOM</text>
+<text x="38.1" y="121.92" size="1.778" layer="94">On BOM</text>
+<text x="175.26" y="228.6" size="1.778" layer="94">On BOM</text>
 <text x="208.28" y="220.98" size="1.778" layer="94" rot="R90">On BOM</text>
-<text x="86.36" y="233.68" size="1.778" layer="94" rot="R90">On BOM</text>
-<text x="35.56" y="228.6" size="1.778" layer="94" rot="R90">On BOM</text>
 <text x="25.4" y="228.6" size="1.778" layer="94" rot="R90">On BOM</text>
 <text x="55.88" y="106.68" size="1.778" layer="94" rot="R90">On BOM</text>
 <text x="17.78" y="139.7" size="1.778" layer="94">On BOM</text>
-<text x="137.16" y="233.68" size="1.778" layer="94" rot="R270">On BOM</text>
 <text x="205.74" y="231.14" size="1.778" layer="94" rot="R90">On BOM</text>
 <text x="243.84" y="236.22" size="1.778" layer="94">On BOM</text>
@@
 <text x="15.24" y="193.04" size="1.778" layer="94" rot="R270">On BOM</text>
 <text x="332.74" y="96.52" size="1.778" layer="94" rot="R270">On BOM</text>
-<text x="135.636" y="222.25" size="1.778" layer="94" rot="R90">On BOM</text>
+<text x="35.56" y="228.6" size="1.778" layer="94" rot="R90">On BOM</text>
+<text x="88.9" y="233.68" size="1.778" layer="94" rot="R90">On BOM</text>
+<text x="66.04" y="238.76" size="1.778" layer="94" rot="R180">On BOM</text>
+<text x="139.7" y="226.06" size="1.778" layer="94" rot="R180">On BOM</text>
+<text x="337.82" y="241.3" size="1.778" layer="94">On BOM</text>
+<text x="309.88" y="142.24" size="1.778" layer="94">On BOM</text>
 </plain>
 <instances>

Commit message: corrected again :-D
now fits box, GSM should fit also
Parts:
- removed U2: ARDUINO, arduino:ARDUINO
- added U3: ARDUINOR3-DIMENSION, adafruit:ARDUINOR3-DIMENSION
Connections:
- net 5VGSM: now also U3.5V; no longer U2.5V
- net GND: now also U3.GND, U3.GND1, U3.GND2; no longer U2.GND, U2.GND1, U2.GND2
- net N$15: now also U3.A1; no longer U2.A1
- net N$19: now also U3.D7; no longer U2.D7
- net N$30: now also U3.D9; no longer U2.D9
- net N$32: now also U3.D8; no longer U2.D8
- net RESET: now also U3./RESET; no longer U2./RESET
- net SCL: now also U3.A5/SCL; no longer U2.A5/SCL
- net SDA: now also U3.A4/SDA; no longer U2.A4/SDA
- net VCC: now also U3.3V; no longer U2.3V
Changed lines of the file:
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@@
 <part name="P+8" library="SparkFun-Aesthetics" deviceset="VCC" device=""/>
 <part name="GND8" library="SparkFun-Aesthetics" deviceset="GND" device=""/>
-<part name="U2" library="arduino" deviceset="ARDUINO" device=""/>
 <part name="GND1" library="SparkFun-Aesthetics" deviceset="GND" device=""/>
 <part name="X1" library="con-wago-500" deviceset="W237-102" device=""/>
@@
 <part name="C5" library="resistor" deviceset="C-EU" device="C0603" value="100nF"/>
 <part name="JP1" library="pinhead" deviceset="PINHD-2X3" device=""/>
+<part name="U3" library="adafruit" deviceset="ARDUINOR3" device="-DIMENSION"/>
 </parts>
 <sheets>
@@
 <instance part="P+8" gate="1" x="256.54" y="246.38"/>
 <instance part="GND8" gate="1" x="251.46" y="223.52"/>
-<instance part="U2" gate="G$1" x="223.52" y="127" rot="R90"/>
 <instance part="GND1" gate="1" x="63.5" y="177.8"/>
 <instance part="X1" gate="-1" x="22.86" y="190.5"/>
@@
 <attribute name="VALUE" x="265.43" y="99.06" size="1.778" layer="96"/>
 </instance>
+<instance part="U3" gate="G$1" x="198.12" y="160.02" rot="R90"/>
 </instances>
 <busses>
@@
 <wire x1="228.6" y1="154.94" x2="233.68" y2="154.94" width="0.1524" layer="91"/>
 <label x="233.68" y="154.94" size="1.778" layer="95"/>
-<pinref part="U2" gate="G$1" pin="3V"/>
+<pinref part="U3" gate="G$1" pin="3V"/>
 </segment>
 <segment>
@@
 </segment>
 <segment>
-<pinref part="U2" gate="G$1" pin="GND1"/>
 <pinref part="GND2" gate="1" pin="GND"/>
 <wire x1="248.92" y1="162.56" x2="228.6" y2="162.56" width="0.1524" layer="91"/>
-<pinref part="U2" gate="G$1" pin="GND2"/>
 <wire x1="228.6" y1="162.56" x2="228.6" y2="160.02" width="0.1524" layer="91"/>
+<pinref part="U3" gate="G$1" pin="GND1"/>
 <junction x="228.6" y="162.56"/>
+<pinref part="U3" gate="G$1" pin="GND2"/>
 </segment>
 <segment>
@@
 </segment>
 <segment>
-<pinref part="U2" gate="G$1" pin="GND"/>
 <pinref part="GND9" gate="1" pin="GND"/>
 <wire x1="157.48" y1="142.24" x2="167.64" y2="142.24" width="0.1524" layer="91"/>
+<pinref part="U3" gate="G$1" pin="GND"/>
 </segment>
 <segment>
@@
 <segment>
 <label x="251.46" y="109.22" size="1.778" layer="95"/>
-<pinref part="U2" gate="G$1" pin="A4/SDA"/>
 <wire x1="228.6" y1="180.34" x2="205.74" y2="180.34" width="0.1524" layer="91"/>
 <wire x1="205.74" y1="180.34" x2="205.74" y2="109.22" width="0.1524" layer="91"/>
@@
 <wire x1="226.06" y1="109.22" x2="248.92" y2="109.22" width="0.1524" layer="91"/>
 <junction x="226.06" y="109.22"/>
+<pinref part="U3" gate="G$1" pin="A4/SDA"/>
 </segment>
 <segment>
@@
 <wire x1="203.2" y1="106.68" x2="203.2" y2="182.88" width="0.1524" layer="91"/>
 <wire x1="203.2" y1="182.88" x2="228.6" y2="182.88" width="0.1524" layer="91"/>
-<pinref part="U2" gate="G$1" pin="A5/SCL"/>
 <pinref part="IC2" gate="1" pin="ANALOG_5"/>
 <junction x="226.06" y="106.68"/>
+<pinref part="U3" gate="G$1" pin="A5/SCL"/>
 </segment>
 <segment>
@@
 <wire x1="236.22" y1="152.4" x2="228.6" y2="152.4" width="0.1524" layer="91"/>
 <label x="238.76" y="152.4" size="1.778" layer="95"/>
-<pinref part="U2" gate="G$1" pin="/RESET"/>
+<pinref part="U3" gate="G$1" pin="/RESET"/>
 </segment>
 <segment>
@@
 <wire x1="226.06" y1="116.84" x2="213.36" y2="116.84" width="0.1524" layer="91"/>
 <wire x1="213.36" y1="116.84" x2="213.36" y2="172.72" width="0.1524" layer="91"/>
-<pinref part="U2" gate="G$1" pin="A1"/>
 <wire x1="213.36" y1="172.72" x2="228.6" y2="172.72" width="0.1524" layer="91"/>
 <pinref part="IC2" gate="1" pin="ANALOG_1"/>
+<pinref part="U3" gate="G$1" pin="A1"/>
 </segment>
 </net>
@@
 <wire x1="190.5" y1="162.56" x2="167.64" y2="162.56" width="0.1524" layer="91"/>
 <wire x1="195.58" y1="73.66" x2="190.5" y2="73.66" width="0.1524" layer="91"/>
-<pinref part="U2" gate="G$1" pin="D7"/>
 <pinref part="R5" gate="G$1" pin="2"/>
+<pinref part="U3" gate="G$1" pin="D7"/>
 </segment>
 </net>
@@
 <wire x1="228.6" y1="157.48" x2="236.22" y2="157.48" width="0.1524" layer="91"/>
 <label x="231.14" y="157.48" size="1.778" layer="95"/>
-<pinref part="U2" gate="G$1" pin="5V"/>
+<pinref part="U3" gate="G$1" pin="5V"/>
 </segment>
 </net>
 <net name="N$30" class="0">
 <segment>
-<pinref part="U2" gate="G$1" pin="D9"/>
 <wire x1="167.64" y1="154.94" x2="182.88" y2="154.94" width="0.1524" layer="91"/>
 <wire x1="182.88" y1="154.94" x2="182.88" y2="106.68" width="0.1524" layer="91"/>
 <pinref part="R17" gate="G$1" pin="1"/>
+<pinref part="U3" gate="G$1" pin="D9"/>
 </segment>
 </net>
 <net name="N$32" class="0">
 <segment>
-<pinref part="U2" gate="G$1" pin="D8"/>
 <wire x1="185.42" y1="157.48" x2="167.64" y2="157.48" width="0.1524" layer="91"/>
 <pinref part="R16" gate="G$1" pin="1"/>
 <wire x1="185.42" y1="124.46" x2="185.42" y2="157.48" width="0.1524" layer="91"/>
-</segment>
-</net>
+<pinref part="U3" gate="G$1" pin="D8"/>
+</segment>
+</net>

Commit message: rev 10 routed
should be good to go
Parts:
- removed U3: ARDUINOR3-DIMENSION, adafruit:ARDUINOR3-DIMENSION
- added U$3: ARDUINO, arduino:ARDUINO
Connections:
- net 5VGSM: now also U$3.5V; no longer U3.5V
- net GND: now also U$3.GND, U$3.GND1, U$3.GND2; no longer U3.GND, U3.GND1, U3.GND2
- net N$15: now also U$3.A1; no longer U3.A1
- net N$19: now also U$3.D7; no longer U3.D7
- net N$30: now also U$3.D9; no longer U3.D9
- net N$32: now also U$3.D8; no longer U3.D8
- net RESET: now also U$3./RESET; no longer U3./RESET
- net SCL: now also U$3.A5/SCL; no longer U3.A5/SCL
- net SDA: now also U$3.A4/SDA; no longer U3.A4/SDA
- net VCC: now also U$3.3V; no longer U3.3V
Changed lines of the file:
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@@
 <part name="C5" library="resistor" deviceset="C-EU" device="C0603" value="100nF"/>
 <part name="JP1" library="pinhead" deviceset="PINHD-2X3" device=""/>
-<part name="U3" library="adafruit" deviceset="ARDUINOR3" device="-DIMENSION"/>
+<part name="U$3" library="arduino" deviceset="ARDUINO" device=""/>
 </parts>
 <sheets>
@@
 <attribute name="VALUE" x="265.43" y="99.06" size="1.778" layer="96"/>
 </instance>
-<instance part="U3" gate="G$1" x="198.12" y="160.02" rot="R90"/>
+<instance part="U$3" gate="G$1" x="223.52" y="127" rot="R90"/>
 </instances>
 <busses>
@@
 <wire x1="228.6" y1="154.94" x2="233.68" y2="154.94" width="0.1524" layer="91"/>
 <label x="233.68" y="154.94" size="1.778" layer="95"/>
-<pinref part="U3" gate="G$1" pin="3V"/>
+<pinref part="U$3" gate="G$1" pin="3V"/>
 </segment>
 <segment>
@@
 <wire x1="248.92" y1="162.56" x2="228.6" y2="162.56" width="0.1524" layer="91"/>
 <wire x1="228.6" y1="162.56" x2="228.6" y2="160.02" width="0.1524" layer="91"/>
-<pinref part="U3" gate="G$1" pin="GND1"/>
+<pinref part="U$3" gate="G$1" pin="GND1"/>
 <junction x="228.6" y="162.56"/>
-<pinref part="U3" gate="G$1" pin="GND2"/>
+<pinref part="U$3" gate="G$1" pin="GND2"/>
 </segment>
 <segment>
@@
 <pinref part="GND9" gate="1" pin="GND"/>
 <wire x1="157.48" y1="142.24" x2="167.64" y2="142.24" width="0.1524" layer="91"/>
-<pinref part="U3" gate="G$1" pin="GND"/>
+<pinref part="U$3" gate="G$1" pin="GND"/>
 </segment>
 <segment>
@@
 <wire x1="226.06" y1="109.22" x2="248.92" y2="109.22" width="0.1524" layer="91"/>
 <junction x="226.06" y="109.22"/>
-<pinref part="U3" gate="G$1" pin="A4/SDA"/>
+<pinref part="U$3" gate="G$1" pin="A4/SDA"/>
 </segment>
 <segment>
@@
 <pinref part="IC2" gate="1" pin="ANALOG_5"/>
 <junction x="226.06" y="106.68"/>
-<pinref part="U3" gate="G$1" pin="A5/SCL"/>
+<pinref part="U$3" gate="G$1" pin="A5/SCL"/>
 </segment>
 <segment>
@@
 <wire x1="236.22" y1="152.4" x2="228.6" y2="152.4" width="0.1524" layer="91"/>
 <label x="238.76" y="152.4" size="1.778" layer="95"/>
-<pinref part="U3" gate="G$1" pin="/RESET"/>
+<pinref part="U$3" gate="G$1" pin="/RESET"/>
 </segment>
 <segment>
@@
 <wire x1="213.36" y1="172.72" x2="228.6" y2="172.72" width="0.1524" layer="91"/>
 <pinref part="IC2" gate="1" pin="ANALOG_1"/>
-<pinref part="U3" gate="G$1" pin="A1"/>
+<pinref part="U$3" gate="G$1" pin="A1"/>
 </segment>
 </net>
@@
 <wire x1="195.58" y1="73.66" x2="190.5" y2="73.66" width="0.1524" layer="91"/>
 <pinref part="R5" gate="G$1" pin="2"/>
-<pinref part="U3" gate="G$1" pin="D7"/>
+<pinref part="U$3" gate="G$1" pin="D7"/>
 </segment>
 </net>
@@
 <wire x1="228.6" y1="157.48" x2="236.22" y2="157.48" width="0.1524" layer="91"/>
 <label x="231.14" y="157.48" size="1.778" layer="95"/>
-<pinref part="U3" gate="G$1" pin="5V"/>
+<pinref part="U$3" gate="G$1" pin="5V"/>
 </segment>
 </net>
@@
 <wire x1="182.88" y1="154.94" x2="182.88" y2="106.68" width="0.1524" layer="91"/>
 <pinref part="R17" gate="G$1" pin="1"/>
-<pinref part="U3" gate="G$1" pin="D9"/>
+<pinref part="U$3" gate="G$1" pin="D9"/>
 </segment>
 </net>
@@
 <pinref part="R16" gate="G$1" pin="1"/>
 <wire x1="185.42" y1="124.46" x2="185.42" y2="157.48" width="0.1524" layer="91"/>
-<pinref part="U3" gate="G$1" pin="D8"/>
-</segment>
-</net>
+<pinref part="U$3" gate="G$1" pin="D8"/>
+</segment>
+</net>

Commit message: rev 10 routed
Connections:
- net N$26: now also I2C_EXT.20; no longer I2C_EXT.5
- net RESET: now also I2C_EXT.5
Other:
- moved on the sheet: C5
Changed lines of the file:
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@@
 <text x="307.34" y="177.8" size="1.778" layer="94" rot="R90">On BOM</text>
 <text x="45.72" y="175.26" size="1.778" layer="94" rot="R180">On BOM</text>
-<text x="121.92" y="195.58" size="1.778" layer="94" rot="R90">On BOM</text>
+<text x="139.7" y="233.68" size="1.778" layer="94" rot="R270">On BOM</text>
 <wire x1="325.12" y1="157.48" x2="325.12" y2="124.46" width="0.3048" layer="94"/>
 <wire x1="325.12" y1="124.46" x2="325.12" y2="83.82" width="0.3048" layer="94"/>
@@
 <instance part="R1" gate="G$1" x="137.16" y="226.06" rot="R270"/>
 <instance part="R3" gate="G$1" x="134.62" y="226.06" rot="R270"/>
-<instance part="C5" gate="G$1" x="121.92" y="200.66" smashed="yes" rot="R180">
-<attribute name="NAME" x="125.476" y="202.819" size="1.778" layer="95" rot="R180"/>
+<instance part="C5" gate="G$1" x="139.7" y="228.6" smashed="yes">
+<attribute name="NAME" x="136.144" y="226.441" size="1.778" layer="95"/>
 </instance>
 <instance part="JP1" gate="A" x="271.78" y="106.68" smashed="yes">
@@
 <segment>
 <pinref part="C5" gate="G$1" pin="1"/>
-<wire x1="121.92" y1="198.12" x2="121.92" y2="190.5" width="0.1524" layer="91"/>
+<wire x1="139.7" y1="231.14" x2="139.7" y2="238.76" width="0.1524" layer="91"/>
+<label x="139.7" y="246.38" size="1.778" layer="95" rot="R270"/>
+</segment>
+<segment>
+<wire x1="121.92" y1="190.5" x2="121.92" y2="210.82" width="0.1524" layer="91"/>
 <label x="121.92" y="187.96" size="1.778" layer="95" rot="R270"/>
+<pinref part="I2C_EXT" gate="A" pin="5"/>
 </segment>
 </net>
@@
 <net name="N$26" class="0">
 <segment>
-<wire x1="121.92" y1="210.82" x2="121.92" y2="205.74" width="0.1524" layer="91"/>
+<pinref part="I2C_EXT" gate="A" pin="20"/>
 <pinref part="C5" gate="G$1" pin="2"/>
-<pinref part="I2C_EXT" gate="A" pin="5"/>
-</segment>
-</net>
+<wire x1="139.7" y1="218.44" x2="139.7" y2="223.52" width="0.1524" layer="91"/>
+</segment>
+</net>

Commit message: fixed rev10 transistor
Parts:
- T1: device transistor:-NPN-SOT23-EBC -> transistor:MMBTH24LT1-NPN-SOT23-BEC
Changed lines of the file:
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@@
 <?xml version="1.0" encoding="utf-8"?>
 <!DOCTYPE eagle SYSTEM "eagle.dtd">
-<eagle version="7.4.0">
+<eagle version="7.5.0">
 <drawing>
 <settings>
@@
 <grid distance="0.1" unitdist="inch" unit="inch" style="lines" multiple="1" display="no" altdistance="0.01" altunitdist="inch" altunit="inch"/>
 <layers>
-<layer number="1" name="Top" color="4" fill="1" visible="no" active="no"/>
-<layer number="16" name="Bottom" color="1" fill="1" visible="no" active="no"/>
-<layer number="17" name="Pads" color="2" fill="1" visible="no" active="no"/>
-<layer number="18" name="Vias" color="2" fill="1" visible="no" active="no"/>
-<layer number="19" name="Unrouted" color="6" fill="1" visible="no" active="no"/>
-<layer number="20" name="Dimension" color="15" fill="1" visible="no" active="no"/>
-<layer number="21" name="tPlace" color="7" fill="1" visible="no" active="no"/>
-<layer number="22" name="bPlace" color="7" fill="1" visible="no" active="no"/>
-<layer number="23" name="tOrigins" color="15" fill="1" visible="no" active="no"/>
-<layer number="24" name="bOrigins" color="15" fill="1" visible="no" active="no"/>
-<layer number="25" name="tNames" color="7" fill="1" visible="no" active="no"/>
-<layer number="26" name="bNames" color="7" fill="1" visible="no" active="no"/>
-<layer number="27" name="tValues" color="7" fill="1" visible="no" active="no"/>
-<layer number="28" name="bValues" color="7" fill="1" visible="no" active="no"/>
+<layer number="1" name="Top" color="4" fill="1" visible="yes" active="no"/>
+<layer number="16" name="Bottom" color="1" fill="1" visible="yes" active="no"/>
+<layer number="17" name="Pads" color="2" fill="1" visible="yes" active="no"/>
+<layer number="18" name="Vias" color="2" fill="1" visible="yes" active="no"/>
+<layer number="19" name="Unrouted" color="6" fill="1" visible="yes" active="no"/>
+<layer number="20" name="Dimension" color="15" fill="1" visible="yes" active="no"/>
+<layer number="21" name="tPlace" color="7" fill="1" visible="yes" active="no"/>
+<layer number="22" name="bPlace" color="7" fill="1" visible="yes" active="no"/>
+<layer number="23" name="tOrigins" color="15" fill="1" visible="yes" active="no"/>
+<layer number="24" name="bOrigins" color="15" fill="1" visible="yes" active="no"/>
+<layer number="25" name="tNames" color="7" fill="1" visible="yes" active="no"/>
+<layer number="26" name="bNames" color="7" fill="1" visible="yes" active="no"/>
+<layer number="27" name="tValues" color="7" fill="1" visible="yes" active="no"/>
+<layer number="28" name="bValues" color="7" fill="1" visible="yes" active="no"/>
 <layer number="29" name="tStop" color="7" fill="3" visible="no" active="no"/>
 <layer number="30" name="bStop" color="7" fill="6" visible="no" active="no"/>
@@
 <layer number="35" name="tGlue" color="7" fill="4" visible="no" active="no"/>
 <layer number="36" name="bGlue" color="7" fill="5" visible="no" active="no"/>
-<layer number="37" name="tTest" color="7" fill="1" visible="no" active="no"/>
-<layer number="38" name="bTest" color="7" fill="1" visible="no" active="no"/>
+<layer number="37" name="tTest" color="7" fill="1" visible="yes" active="no"/>
+<layer number="38" name="bTest" color="7" fill="1" visible="yes" active="no"/>
 <layer number="39" name="tKeepout" color="4" fill="11" visible="no" active="no"/>
 <layer number="40" name="bKeepout" color="1" fill="11" visible="no" active="no"/>
@@
 <layer number="44" name="Drills" color="7" fill="1" visible="no" active="no"/>
 <layer number="45" name="Holes" color="7" fill="1" visible="no" active="no"/>
-<layer number="46" name="Milling" color="3" fill="1" visible="no" active="no"/>
-<layer number="47" name="Measures" color="7" fill="1" visible="no" active="no"/>
-<layer number="48" name="Document" color="7" fill="1" visible="no" active="no"/>
-<layer number="49" name="Reference" color="7" fill="1" visible="no" active="no"/>
-<layer number="50" name="dxf" color="7" fill="1" visible="no" active="no"/>
-<layer number="51" name="tDocu" color="7" fill="1" visible="no" active="no"/>
-<layer number="52" name="bDocu" color="7" fill="1" visible="no" active="no"/>
-<layer number="53" name="tGND_GNDA" color="7" fill="9" visible="no" active="no"/>
-<layer number="54" name="bGND_GNDA" color="1" fill="9" visible="no" active="no"/>
-<layer number="56" name="wert" color="7" fill="1" visible="no" active="no"/>
-<layer number="57" name="tCAD" color="7" fill="1" visible="no" active="no"/>
+<layer number="46" name="Milling" color="3" fill="1" visible="yes" active="no"/>
+<layer number="47" name="Measures" color="7" fill="1" visible="yes" active="no"/>
+<layer number="48" name="Document" color="7" fill="1" visible="yes" active="no"/>
+<layer number="49" name="Reference" color="7" fill="1" visible="yes" active="no"/>
+<layer number="50" name="dxf" color="7" fill="1" visible="yes" active="no"/>
+<layer number="51" name="tDocu" color="7" fill="1" visible="yes" active="no"/>
+<layer number="52" name="bDocu" color="7" fill="1" visible="yes" active="no"/>
+<layer number="53" name="tGND_GNDA" color="7" fill="9" visible="yes" active="no"/>
+<layer number="54" name="bGND_GNDA" color="1" fill="9" visible="yes" active="no"/>
+<layer number="56" name="wert" color="7" fill="1" visible="yes" active="no"/>
+<layer number="57" name="tCAD" color="7" fill="1" visible="yes" active="no"/>
 <layer number="90" name="Modules" color="5" fill="1" visible="yes" active="yes"/>
 <layer number="91" name="Nets" color="2" fill="1" visible="yes" active="yes"/>
@@
 <part name="R11" library="resistor" deviceset="R-EU_" device="R0603" value="470R"/>
 <part name="LED1" library="led" deviceset="LED" device="CHIP-LED0603"/>
-<part name="T1" library="transistor" deviceset="*-NPN-" device="SOT23-EBC"/>
+<part name="T1" library="transistor" deviceset="*-NPN-" device="SOT23-BEC" technology="MMBTH24LT1"/>
 <part name="R13" library="resistor" deviceset="R-EU_" device="R0603" value="1K"/>
 <part name="R14" library="resistor" deviceset="R-EU_" device="R0603" value="10K"/>
