File: Arduino/hardware/proposed/building blocks/AVR.sch (EAGLE design)
At the start: 36 parts, among them IC1 LTC3525, IC2 ATMEGA168-AU, Q1 32768Hz, U1 RN2483, U2 TMP112, X1 SMA-142-0701-881/886, X2 SMA-142-0701-881/886

Commit message: reservered space for mobdet on rev 14
Parts:
- removed +, -: (no value), wirepad:2,15/1,0
- removed C1: 1µ, SparkFun:CAP0603-CAP
- removed C11: 100nF, resistor:C-EUC0603
- removed C2: 10µ, SparkFun:CAP0805
- removed C4: 100n, rcl:C-EUC0603
- removed FTDI_RN2483: (no value), pinhead:PINHD-1X6
- removed IC1: LTC3525, JeeLabs:LTC3525
- removed JP1: (no value), pinhead:PINHD-1X1
- removed JP2: (no value), pinhead:PINHD-1X2
- removed JP3: (no value), pinhead:PINHD-1X3
- removed L1: 10 µH, SparkFun:INDUCTOR1210
- removed PHT: BPX65, opto-trans-siemens:BPX65
- removed R1: 100K, resistor:R-EU_R0603
- removed R10, R11, R5, R7: 4.7K, resistor:R-EU_R0603
- removed U1: RN2483, RFM95W-RN2483:RN2483
- removed U2: TMP112, TMP112_2:TMP112
- removed X1, X2: SMA-142-0701-881/886, con-coax:SMA-142-0701-881/886
- added PAD1, PAD10, PAD11, PAD12, PAD13, PAD14, PAD15, PAD16, PAD17, PAD18, PAD19, PAD2, PAD20, PAD21, PAD22, PAD23, PAD24, PAD25, PAD3, PAD4, PAD5, PAD6, PAD7, PAD8, PAD9: (no value), wirepad:1,6/0,8
Connections:
- removed net CHG_PUMP: IC1.SHDN
- removed net LDR: IC2.ANALOG_0, PHT.C, R1.1
- removed net N$22: U1.RFH, X1.1
- removed net N$33: U1.RFL, X2.1
- removed net PHONE: IC2.ANALOG_1
- removed net RN2483_RESET: C11.1, U1.RESET
- removed net RN2483_UART_CTS: FTDI_RN2483.2, U1.UART_CTS
- removed net RN2483_UART_RTS: IC2.ANALOG_7, U1.UART_RTS
- removed net RN2483_UART_RX: R10.1, R5.1, U1.UART_RX
- removed net RN2483_UART_TX: R11.1, R7.1, U1.UART_TX
- removed net VCC1: C2.1, IC1.VOUT, JP3.1
- removed net VOICE_NIRQ: IC2.DIGITAL_6(PWM), JP1.1
- new net N$11: IC2.DIGITAL_5(PWM), PAD17.P
- new net N$12: IC2.DIGITAL_6(PWM), PAD18.P
- new net N$13: IC2.DIGITAL_7, PAD19.P
- new net N$14: IC2.ANALOG_3, PAD7.P
- new net N$15: IC2.ANALOG_7, PAD11.P
- new net N$16: IC2.DIGITAL_8, PAD20.P
- net D2: now also PAD14.P
- net GND: now also PAD2.P; no longer -.P, C1.2, C2.2, C4.2, FTDI_RN2483.1, IC1.GND1, IC1.GND2, JP3.3, R1.2, U1.GND@1, U1.GND@10, U1.GND@11, U1.GND@12, U1.GND@13, U1.GND@2, U1.GND@3, U1.GND@4, U1.GND@5, U1.GND@6, U1.GND@7, U1.GND@8, U1.GND@9, U2.ADD0, U2.GND, X1.2, X2.2
- net IO_POWER_UP: no longer IC2.DIGITAL_7, PHT.A
- net N$10: now also IC2.DIGITAL_4, PAD16.P; no longer IC1.SW, L1.2
- net N$2: now also IC2.ANALOG_0, PAD4.P; no longer C11.2, FTDI_RN2483.6
- net N$5: now also IC2.ANALOG_1, PAD5.P; no longer FTDI_RN2483.4, R7.2
- net N$7: now also IC2.ANALOG_2, PAD6.P; no longer FTDI_RN2483.5, R5.2
- net N$8: now also IC2.ANALOG_6, PAD10.P; no longer IC2.DIGITAL_5(PWM), R10.2
- net N$9: now also IC2.DIGITAL_3(PWM), PAD15.P; no longer IC2.DIGITAL_8, R11.2
- net RESET: now also PAD1.P
- net RFM_IRQ: now also PAD21.P
- net RX: now also PAD13.P
- net SCL: now also PAD9.P; no longer JP2.2, U2.SCL
- net SDA: now also PAD8.P; no longer JP2.1, U2.SDA
- net SPI_MISO: now also PAD24.P
- net SPI_MOSI: now also PAD23.P
- net SPI_NSS: now also PAD22.P
- net SPI_SCK: now also PAD25.P
- net TX: now also PAD12.P
- net VCC: now also PAD3.P; no longer +.P, C1.1, C4.1, FTDI_RN2483.3, IC1.VIN, L1.1, U1.3.3V, U1.3.3V@1, U2.V+
Other:
- note added: "I2C Pullup's"
- note removed: "Battery Connection"
- note removed: "Charge Pump"
- note removed: "Light Sensor"
- note removed: "LoRa MODULE"
- note removed: "Programming for LoRa MODULE"
- note removed: "TMP112 + I2C Pullup's"
- note removed: "VOICE MODULE"
- moved on the sheet: R6, R8
