File: Arduino/hardware/REV14/REV14.brd (EAGLE design)
At the start: 100 x 50 mm, 45 parts, among them IC1 LTC3525, IC2 ATMEGA168-AU, Q1 32768Hz, U1 RN2483, U2 TMP112

Commit message: rev14 with mobile detect
Parts:
- added C13: 0.1uF, resistor:C0603
- added C3, C6: 22pF, resistor:C0603
- added C7: 0.22uF, resistor:C0603
- added C8: 100uF, resistor:C0603
- added IC3: TS1003IG5TMF, TS1003IG5T:TS1003IG5T
- added PAD1: (no value), wirepad:2,15/1,0
- added R19, R21: 2.2M, resistor:R0603
- added R20: 100K, resistor:R0603
Connections:
- new net N$18: C3.1, PAD1.1
- new net N$19: C3.2, C6.1, C7.2, IC3.4, R21.1
- new net N$21: C7.1, C8.1, IC3.3, R19.2, R20.1
- net GND: now also C13.2, C6.2, C8.2, IC3.2, R20.2
- net PHONE: now also C13.1, IC3.1, R21.2
- net VCC: now also IC3.5, R19.1
Changed lines of the file:
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@@
 </element>
 <element name="R15" library="resistor" package="R0603" value="4.7K" x="25.7175" y="34.925" smashed="yes">
-<attribute name="NAME" x="24.8285" y="35.814" size="1.27" layer="25"/>
+<attribute name="NAME" x="24.8285" y="35.814" size="1" layer="25"/>
 </element>
 <element name="R17" library="resistor" package="R0603" value="4.7K" x="17.4625" y="8.5725" smashed="yes">
-<attribute name="NAME" x="16.5735" y="9.4615" size="1.27" layer="25"/>
+<attribute name="NAME" x="16.5735" y="9.4615" size="1" layer="25"/>
 </element>
 <element name="R18" library="resistor" package="R0603" value="4.7K" x="86.995" y="12.065" smashed="yes" rot="R270">
-<attribute name="NAME" x="86.106" y="13.9065" size="1.27" layer="25"/>
+<attribute name="NAME" x="86.106" y="13.9065" size="1" layer="25"/>
+</element>
+<element name="IC3" library="TS1003IG5T" package="TS1003IG5T" value="TS1003IG5TMF" x="95.25" y="27.94" smashed="yes">
+<attribute name="NAME" x="93.472" y="26.162" size="1" layer="25" ratio="10" rot="R90"/>
+</element>
+<element name="C3" library="resistor" package="C0603" value="22pF" x="97.79" y="33.02" smashed="yes" rot="R180">
+<attribute name="NAME" x="98.679" y="35.433" size="1" layer="25" rot="R180"/>
+</element>
+<element name="C6" library="resistor" package="C0603" value="22pF" x="92.71" y="33.02" smashed="yes" rot="R180">
+<attribute name="NAME" x="93.599" y="32.258" size="1" layer="25" rot="R180"/>
+</element>
+<element name="C7" library="resistor" package="C0603" value="0.22uF" x="96.52" y="21.59" smashed="yes" rot="R180">
+<attribute name="NAME" x="97.409" y="20.828" size="1" layer="25" rot="R180"/>
+</element>
+<element name="C8" library="resistor" package="C0603" value="100uF" x="90.17" y="27.94" smashed="yes" rot="R90">
+<attribute name="NAME" x="89.408" y="27.051" size="1" layer="25" rot="R90"/>
+</element>
+<element name="R19" library="resistor" package="R0603" value="2.2M" x="88.9" y="35.56" smashed="yes" rot="R180">
+<attribute name="NAME" x="89.789" y="34.671" size="1" layer="25" rot="R180"/>
+</element>
+<element name="R20" library="resistor" package="R0603" value="100K" x="83.82" y="31.75" smashed="yes" rot="R270">
+<attribute name="NAME" x="84.709" y="32.639" size="1" layer="25" rot="R270"/>
+</element>
+<element name="R21" library="resistor" package="R0603" value="2.2M" x="90.17" y="21.59" smashed="yes" rot="R90">
+<attribute name="NAME" x="89.281" y="20.701" size="1" layer="25" rot="R90"/>
+</element>
+<element name="C13" library="resistor" package="C0603" value="0.1uF" x="83.82" y="25.4" smashed="yes" rot="R90">
+<attribute name="NAME" x="83.058" y="24.511" size="1" layer="25" rot="R90"/>
+</element>
+<element name="PAD1" library="wirepad" package="2,15/1,0" value="" x="98.425" y="27.94" smashed="yes">
+<attribute name="VALUE" x="98.425" y="28.94" size="0.0254" layer="27"/>
 </element>
 </elements>
@@
 <contactref element="R17" pad="2"/>
 <contactref element="R18" pad="1"/>
+<contactref element="C6" pad="2"/>
+<contactref element="R20" pad="2"/>
+<contactref element="C8" pad="2"/>
+<contactref element="C13" pad="2"/>
+<contactref element="IC3" pad="2"/>
 <wire x1="81.5975" y1="45.4025" x2="93.345" y2="45.4025" width="0" layer="19" extent="1-1"/>
+<wire x1="83.82" y1="30.9" x2="81.4375" y2="41.97" width="0" layer="19" extent="1-1"/>
+<wire x1="83.82" y1="26.25" x2="83.82" y2="30.9" width="0" layer="19" extent="1-1"/>
+<wire x1="90.17" y1="28.79" x2="83.82" y2="30.9" width="0" layer="19" extent="1-1"/>
+<wire x1="91.86" y1="33.02" x2="90.17" y2="28.79" width="0" layer="19" extent="1-1"/>
+<wire x1="95.25" y1="26.634" x2="90.17" y2="28.79" width="0" layer="19" extent="1-1"/>
+<wire x1="86.995" y1="12.915" x2="83.82" y2="26.25" width="0" layer="19" extent="1-1"/>
+<wire x1="86.36" y1="4.635" x2="86.995" y2="12.915" width="0" layer="19" extent="1-1"/>
+<wire x1="91.44" y1="4.635" x2="86.36" y2="4.635" width="0" layer="19" extent="1-1"/>
 <wire x1="61.055" y1="38.325" x2="81.4375" y2="41.97" width="0" layer="19" extent="1-1"/>
 <wire x1="58.1025" y1="36.64" x2="58.6025" y2="38.29" width="0" layer="19" extent="1-1"/>
@@
 <wire x1="15.715" y1="16.6025" x2="19.525" y2="21.6825" width="0" layer="19" extent="1-1"/>
 <wire x1="19.525" y1="12.7925" x2="15.715" y2="16.6025" width="0" layer="19" extent="1-1"/>
-<wire x1="18.5075" y1="6.795" x2="19.525" y2="12.7925" width="0" layer="19" extent="1-1"/>
+<wire x1="18.3125" y1="8.5725" x2="19.525" y2="12.7925" width="0" layer="19" extent="1-1"/>
+<wire x1="18.5075" y1="6.795" x2="18.3125" y2="8.5725" width="0" layer="19" extent="1-1"/>
 <wire x1="9.365" y1="14.0625" x2="15.715" y2="16.6025" width="0" layer="19" extent="1-1"/>
 <wire x1="5.8725" y1="12.7925" x2="9.365" y2="14.0625" width="0" layer="19" extent="1-1"/>
@@
 <wire x1="54.61" y1="6.35" x2="56.5125" y2="17.145" width="0" layer="19" extent="1-1"/>
 <wire x1="35.56" y1="5.5" x2="35.8775" y2="17.085" width="0" layer="19" extent="1-1"/>
-<wire x1="18.3125" y1="8.5725" x2="18.415" y2="3.4925" width="0" layer="19" extent="1-1"/>
-<wire x1="86.995" y1="12.915" x2="18.3125" y2="8.5725" width="0" layer="19" extent="1-1"/>
-<wire x1="86.36" y1="4.635" x2="60.3225" y2="20.0025" width="0" layer="19" extent="1-1"/>
-<wire x1="91.44" y1="4.635" x2="86.36" y2="4.635" width="0" layer="19" extent="1-1"/>
 </signal>
 <signal name="VCC" class="1">
@@
 <contactref element="JP4" pad="4"/>
 <contactref element="R15" pad="1"/>
+<contactref element="R19" pad="1"/>
+<contactref element="IC3" pad="5"/>
 <wire x1="58.1025" y1="42.249071875" x2="90.805" y2="45.4025" width="0" layer="19" extent="1-1"/>
 <wire x1="47.205" y1="27.07" x2="52.07" y2="21.47" width="0" layer="19" extent="1-1"/>
@@
 <wire x1="36.1" y1="22.3774" x2="36.9" y2="30.9626" width="0" layer="19" extent="1-1"/>
 <wire x1="24.8675" y1="26.67" x2="36.1" y2="22.3774" width="0" layer="19" extent="1-1"/>
+<wire x1="24.8675" y1="34.925" x2="24.85" y2="26.6875" width="0" layer="19" extent="1-1"/>
 <wire x1="79.375" y1="12.915" x2="59.69" y2="6.35" width="0" layer="19" extent="1-1"/>
 <wire x1="96.52" y1="4.635" x2="79.375" y2="12.915" width="0" layer="19" extent="1-1"/>
-<wire x1="24.8675" y1="34.925" x2="13.335" y2="25.7175" width="0" layer="19" extent="1-1"/>
+<wire x1="94.3" y1="29.246" x2="3.9475" y2="29.2275" width="0" layer="19" extent="1-1"/>
+<wire x1="89.75" y1="35.56" x2="94.3" y2="29.246" width="0" layer="19" extent="1-1"/>
 </signal>
 <signal name="SPI_SCK">
@@
 <contactref element="IC2" pad="24"/>
 <contactref element="R16" pad="2"/>
-<wire x1="94.4" y1="40.64" x2="40.9" y2="22.3774" width="0" layer="19" extent="1-1"/>
+<contactref element="IC3" pad="1"/>
+<contactref element="R21" pad="2"/>
+<contactref element="C13" pad="1"/>
+<wire x1="40.9" y1="22.3774" x2="94.4" y2="40.64" width="0" layer="19" extent="1-1"/>
+<wire x1="94.3" y1="26.634" x2="40.9" y2="22.3774" width="0" layer="19" extent="1-1"/>
+<wire x1="90.17" y1="22.44" x2="94.3" y2="26.634" width="0" layer="19" extent="1-1"/>
+<wire x1="83.82" y1="24.55" x2="90.17" y2="22.44" width="0" layer="19" extent="1-1"/>
 </signal>
 <signal name="N$11">
@@
 <wire x1="86.995" y1="11.215" x2="83.82" y2="4.635" width="0" layer="19" extent="1-1"/>
 </signal>
+<signal name="N$18">
+<contactref element="PAD1" pad="1"/>
+<contactref element="C3" pad="1"/>
+<wire x1="98.64" y1="33.02" x2="98.425" y2="27.94" width="0" layer="19" extent="1-1"/>
+</signal>
+<signal name="N$19">
+<contactref element="C3" pad="2"/>
+<contactref element="C6" pad="1"/>
+<contactref element="C7" pad="2"/>
+<contactref element="IC3" pad="4"/>
+<contactref element="R21" pad="1"/>
+<wire x1="95.67" y1="21.59" x2="90.17" y2="20.74" width="0" layer="19" extent="1-1"/>
+<wire x1="93.56" y1="33.02" x2="95.67" y2="21.59" width="0" layer="19" extent="1-1"/>
+<wire x1="96.94" y1="33.02" x2="93.56" y2="33.02" width="0" layer="19" extent="1-1"/>
+<wire x1="96.2" y1="29.246" x2="96.94" y2="33.02" width="0" layer="19" extent="1-1"/>
+</signal>
+<signal name="N$21">
+<contactref element="C8" pad="1"/>
+<contactref element="R20" pad="1"/>
+<contactref element="C7" pad="1"/>
+<contactref element="R19" pad="2"/>
+<contactref element="IC3" pad="3"/>
+<wire x1="88.05" y1="35.56" x2="83.82" y2="32.6" width="0" layer="19" extent="1-1"/>
+<wire x1="90.17" y1="27.09" x2="88.05" y2="35.56" width="0" layer="19" extent="1-1"/>
+<wire x1="97.37" y1="21.59" x2="90.17" y2="27.09" width="0" layer="19" extent="1-1"/>
+<wire x1="96.2" y1="26.634" x2="97.37" y2="21.59" width="0" layer="19" extent="1-1"/>
+</signal>
 </signals>

Commit message: rev14 routed
Parts:
- C7: device resistor:C0603 -> rcl:C050H075X075
- moved C7 7.86 mm to (91.1, 27.3), turned to 90 degrees
- moved C8 2.62 mm to (87.6, 27.3)
- moved R15 0.64 mm to (25.7, 35.6), turned to 180 degrees
Routing:
- net VCC: track 100.3 -> 231.3 mm
- net SPI_MOSI: track 0.00 -> 90.1 mm, vias 0 -> 2
- net PHONE: track 0.00 -> 83.0 mm, vias 0 -> 5
- net SPI_MISO: track 0.00 -> 81.9 mm, vias 0 -> 3
- net RFM_IRQ: track 0.00 -> 74.2 mm, vias 0 -> 2
- net SCL: track 19.2 -> 93.2 mm, vias 2 -> 4
- net SDA: track 25.9 -> 95.6 mm, vias 2 -> 5
- net SPI_SCK: track 0.00 -> 66.7 mm, vias 0 -> 3
- net RESET: track 3.11 -> 66.6 mm, vias 0 -> 2
- net D2: track 0.00 -> 61.7 mm
- net VCC1: track 2.53 -> 62.8 mm
- net IO_POWER_UP: track 0.00 -> 60.3 mm, vias 0 -> 1
- net SPI_NSS: track 0.00 -> 55.9 mm, vias 0 -> 3
- net TX: track 0.00 -> 49.9 mm, vias 0 -> 2
- net RX: track 0.00 -> 46.5 mm, vias 0 -> 2
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
Commit message: rev 14 ready for gerbers
Parts:
- removed TP2: TPB1,27, testpad:B1,27
- added PAD2, PAD3: (no value), wirepad:3,81/1,4
- added TP4: TPSQTP06R, testpad:TP06R
Connections:
- net N$22: now also PAD3.1
- net N$33: now also PAD2.1, TP4.TP; no longer TP2.TP
Routing:
- net N$150: track 11.9 -> 0.00 mm, vias 2 -> 0
- net SCL: track 93.2 -> 95.6 mm
- net GND: track 59.0 -> 58.0 mm, vias 129 -> 128
- net N$33: track 156.1 -> 155.2 mm
