File: Arduino/hardware/REV14/REV14.sch (EAGLE design)
At the start: 57 parts, among them IC1 LTC3525, IC2 ATMEGA168-AU, IC3 TS1003IG5TMF, Q1 32768Hz, U1 RN2483, U2 TMP112

Commit message: rev14 pre routing.... again :-D
Parts:
- removed PAD2, PAD3: (no value), wirepad:3,81/1,4
- removed TP4: TPSQTP06R, testpad:TPSQTP06R
- added TP3: TPSQTP07R, testpad:TPSQTP07R
Connections:
- net N$22: no longer PAD3.P
- net N$33: now also TP3.TP; no longer PAD2.P, TP4.TP
Changed lines of the file:
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@@
 </variantdefs>
 <classes>
-<class number="0" name="default" width="0.2032" drill="0">
+<class number="0" name="default" width="0.2032" drill="0.5">
 </class>
-<class number="1" name="supply" width="0.4" drill="0">
+<class number="1" name="supply" width="0.4" drill="0.5">
 <clearance class="1" value="0.2032"/>
 </class>
-<class number="2" name="ant" width="2.1844" drill="0">
+<class number="2" name="ant" width="2.1844" drill="0.5">
 </class>
 </classes>
@@
 <part name="P+6" library="SparkFun-Aesthetics" deviceset="VCC" device=""/>
 <part name="GND9" library="SparkFun-Aesthetics" deviceset="GND" device=""/>
-<part name="PAD2" library="wirepad" deviceset="3,81/1,4" device=""/>
-<part name="PAD3" library="wirepad" deviceset="3,81/1,4" device=""/>
-<part name="TP4" library="testpad" deviceset="TPSQ" device="TP06R"/>
+<part name="TP3" library="testpad" deviceset="TPSQ" device="TP07R"/>
 </parts>
 <sheets>
@@
 <instance part="P+6" gate="G$1" x="40.64" y="71.12"/>
 <instance part="GND9" gate="1" x="63.5" y="43.18"/>
-<instance part="PAD2" gate="1" x="327.66" y="246.38" rot="R270"/>
-<instance part="PAD3" gate="1" x="337.82" y="241.3" rot="R180"/>
-<instance part="TP4" gate="G$1" x="317.5" y="241.3"/>
+<instance part="TP3" gate="G$1" x="322.58" y="246.38" rot="R180"/>
 </instances>
 <busses>
@@
 <wire x1="228.6" y1="205.74" x2="218.44" y2="205.74" width="0.1524" layer="91"/>
 <pinref part="U$4" gate="G$1" pin="V+"/>
-<label x="213.36" y="205.74" size="1.778" layer="95"/>
 </segment>
 <segment>
@@
 <wire x1="254" y1="198.12" x2="259.08" y2="198.12" width="0.1524" layer="91"/>
 <pinref part="U$4" gate="G$1" pin="SDA"/>
-<label x="256.54" y="195.58" size="1.778" layer="95"/>
 </segment>
 </net>
@@
 <wire x1="218.44" y1="198.12" x2="228.6" y2="198.12" width="0.1524" layer="91"/>
 <pinref part="U$4" gate="G$1" pin="SCL"/>
-<label x="213.36" y="198.12" size="1.778" layer="95"/>
 </segment>
 </net>
@@
 <segment>
 <pinref part="U1" gate="G$1" pin="RFH"/>
-<wire x1="335.28" y1="226.06" x2="335.28" y2="241.3" width="0.1524" layer="91"/>
+<wire x1="335.28" y1="226.06" x2="335.28" y2="243.84" width="0.1524" layer="91"/>
 <pinref part="TP1" gate="G$1" pin="TP"/>
-<pinref part="PAD3" gate="1" pin="P"/>
-<wire x1="335.28" y1="241.3" x2="335.28" y2="243.84" width="0.1524" layer="91"/>
-<junction x="335.28" y="241.3"/>
 </segment>
 </net>
@@
 <wire x1="330.2" y1="226.06" x2="330.2" y2="241.3" width="0.1524" layer="91"/>
 <wire x1="330.2" y1="241.3" x2="327.66" y2="243.84" width="0.1524" layer="91"/>
-<wire x1="327.66" y1="243.84" x2="317.5" y2="243.84" width="0.1524" layer="91"/>
-<pinref part="PAD2" gate="1" pin="P"/>
-<junction x="327.66" y="243.84"/>
-<pinref part="TP4" gate="G$1" pin="TP"/>
-</segment>
-</net>
+<wire x1="327.66" y1="243.84" x2="322.58" y2="243.84" width="0.1524" layer="91"/>
+<pinref part="TP3" gate="G$1" pin="TP"/>
+</segment>
+</net>

Commit message: rev14 routed again
Parts:
- added PAD2, PAD3: (no value), wirepad:3,81/1,4
Connections:
- net N$22: now also PAD2.P
- net N$33: now also PAD3.P
Changed lines of the file:
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@@
 <part name="GND9" library="SparkFun-Aesthetics" deviceset="GND" device=""/>
 <part name="TP3" library="testpad" deviceset="TPSQ" device="TP07R"/>
+<part name="PAD2" library="wirepad" deviceset="3,81/1,4" device=""/>
+<part name="PAD3" library="wirepad" deviceset="3,81/1,4" device=""/>
 </parts>
 <sheets>
@@
 <instance part="GND9" gate="1" x="63.5" y="43.18"/>
 <instance part="TP3" gate="G$1" x="322.58" y="246.38" rot="R180"/>
+<instance part="PAD2" gate="1" x="337.82" y="241.3" rot="R180"/>
+<instance part="PAD3" gate="1" x="327.66" y="241.3"/>
 </instances>
 <busses>
@@
 <segment>
 <pinref part="U1" gate="G$1" pin="RFH"/>
-<wire x1="335.28" y1="226.06" x2="335.28" y2="243.84" width="0.1524" layer="91"/>
+<wire x1="335.28" y1="226.06" x2="335.28" y2="241.3" width="0.1524" layer="91"/>
 <pinref part="TP1" gate="G$1" pin="TP"/>
+<pinref part="PAD2" gate="1" pin="P"/>
+<wire x1="335.28" y1="241.3" x2="335.28" y2="243.84" width="0.1524" layer="91"/>
+<junction x="335.28" y="241.3"/>
 </segment>
 </net>
@@
 <wire x1="327.66" y1="243.84" x2="322.58" y2="243.84" width="0.1524" layer="91"/>
 <pinref part="TP3" gate="G$1" pin="TP"/>
-</segment>
-</net>
+<pinref part="PAD3" gate="1" pin="P"/>
+<junction x="330.2" y="241.3"/>
+</segment>
+</net>
