File: Arduino/hardware/REV14/REV14.sch (EAGLE design)
At the start: 57 parts, among them IC1 LTC3525, IC2 ATMEGA168-AU, IC3 TS1003IG5TMF, Q1 32768Hz, U1 RN2483, U2 TMP112

Commit message: fixed cap footprint for mobile detect
Parts:
- C8: device resistor:C-EUC0603 -> rcl:C-EUC1206
Changed lines of the file:
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@@
 <part name="C6" library="resistor" deviceset="C-EU" device="C0603" value="22pF"/>
 <part name="C7" library="rcl" deviceset="C-EU" device="050H075X075" value="0.22uF"/>
-<part name="C8" library="resistor" deviceset="C-EU" device="C0603" value="100uF"/>
+<part name="C8" library="rcl" deviceset="C-EU" device="C1206" value="100uF"/>
 <part name="R19" library="resistor" deviceset="R-EU_" device="R0603" value="2.2M"/>
 <part name="R20" library="resistor" deviceset="R-EU_" device="R0603" value="100K"/>

Commit message: rev14 cut2
Parts:
- removed JP1: (no value), pinhead:PINHD-1X1
- JP2: device pinhead:PINHD-1X2 -> pinhead:PINHD-1X10
- JP3: device pinhead:PINHD-1X3 -> pinhead:PINHD-1X6
- PAD2, PAD3: device wirepad:3,81/1,4 -> wirepad:2,15/1,0
Connections:
- net RN2483_UART_RX: now also R7.1; no longer R5.1
- net RN2483_UART_TX: now also R5.1; no longer R7.1
- net VOICE_NIRQ: now also JP2.8; no longer JP1.1
Other:
- note added: "Copyright and related rights are licensed under the Solderpad Hardware License,"
- note added: "OF ANY KIND, either express or implied. See the Licence for the"
- note added: "Unless required by applicable law or agreed to in writing,"
- note added: "Version 0.51 (the "Licence"); you may not use this file except in compliance"
- note added: "http://solderpad.org/licenses/SHL-0.51."
- note added: "is distributed on an "AS IS" BASIS, WITHOUT WARRANTIES OR CONDITIONS"
- note added: "software, hardware and materials distributed under this Licence"
- note added: "specific language governing permissions and limitations under the Licence."
- note added: "with the Licence. You may obtain a copy of the Licence at"

Commit message: rev14 cut2 corrected
Connections:
- net GND: now also JP3.1; no longer JP3.3
- net SCL: now also JP2.1; no longer JP2.2
- net SDA: now also JP2.2; no longer JP2.1
- net VCC1: now also JP3.3; no longer JP3.1
Changed lines of the file:
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@@
 <grid distance="0.1" unitdist="inch" unit="inch" style="lines" multiple="1" display="no" altdistance="0.01" altunitdist="inch" altunit="inch"/>
 <layers>
-<layer number="1" name="Top" color="4" fill="1" visible="yes" active="no"/>
-<layer number="16" name="Bottom" color="1" fill="1" visible="yes" active="no"/>
-<layer number="17" name="Pads" color="2" fill="1" visible="yes" active="no"/>
-<layer number="18" name="Vias" color="2" fill="1" visible="yes" active="no"/>
-<layer number="19" name="Unrouted" color="6" fill="1" visible="yes" active="no"/>
-<layer number="20" name="Dimension" color="15" fill="1" visible="yes" active="no"/>
-<layer number="21" name="tPlace" color="7" fill="1" visible="yes" active="no"/>
-<layer number="22" name="bPlace" color="7" fill="1" visible="yes" active="no"/>
-<layer number="23" name="tOrigins" color="15" fill="1" visible="yes" active="no"/>
-<layer number="24" name="bOrigins" color="15" fill="1" visible="yes" active="no"/>
-<layer number="25" name="tNames" color="7" fill="1" visible="yes" active="no"/>
-<layer number="26" name="bNames" color="7" fill="1" visible="yes" active="no"/>
-<layer number="27" name="tValues" color="7" fill="1" visible="yes" active="no"/>
-<layer number="28" name="bValues" color="7" fill="1" visible="yes" active="no"/>
+<layer number="1" name="Top" color="4" fill="1" visible="no" active="no"/>
+<layer number="16" name="Bottom" color="1" fill="1" visible="no" active="no"/>
+<layer number="17" name="Pads" color="2" fill="1" visible="no" active="no"/>
+<layer number="18" name="Vias" color="2" fill="1" visible="no" active="no"/>
+<layer number="19" name="Unrouted" color="6" fill="1" visible="no" active="no"/>
+<layer number="20" name="Dimension" color="15" fill="1" visible="no" active="no"/>
+<layer number="21" name="tPlace" color="7" fill="1" visible="no" active="no"/>
+<layer number="22" name="bPlace" color="7" fill="1" visible="no" active="no"/>
+<layer number="23" name="tOrigins" color="15" fill="1" visible="no" active="no"/>
+<layer number="24" name="bOrigins" color="15" fill="1" visible="no" active="no"/>
+<layer number="25" name="tNames" color="7" fill="1" visible="no" active="no"/>
+<layer number="26" name="bNames" color="7" fill="1" visible="no" active="no"/>
+<layer number="27" name="tValues" color="7" fill="1" visible="no" active="no"/>
+<layer number="28" name="bValues" color="7" fill="1" visible="no" active="no"/>
 <layer number="29" name="tStop" color="7" fill="3" visible="no" active="no"/>
 <layer number="30" name="bStop" color="7" fill="6" visible="no" active="no"/>
@@
 <layer number="35" name="tGlue" color="7" fill="4" visible="no" active="no"/>
 <layer number="36" name="bGlue" color="7" fill="5" visible="no" active="no"/>
-<layer number="37" name="tTest" color="7" fill="1" visible="yes" active="no"/>
-<layer number="38" name="bTest" color="7" fill="1" visible="yes" active="no"/>
+<layer number="37" name="tTest" color="7" fill="1" visible="no" active="no"/>
+<layer number="38" name="bTest" color="7" fill="1" visible="no" active="no"/>
 <layer number="39" name="tKeepout" color="4" fill="11" visible="no" active="no"/>
 <layer number="40" name="bKeepout" color="1" fill="11" visible="no" active="no"/>
@@
 <layer number="44" name="Drills" color="7" fill="1" visible="no" active="no"/>
 <layer number="45" name="Holes" color="7" fill="1" visible="no" active="no"/>
-<layer number="46" name="Milling" color="3" fill="1" visible="yes" active="no"/>
-<layer number="47" name="Measures" color="7" fill="1" visible="yes" active="no"/>
-<layer number="48" name="Document" color="7" fill="1" visible="yes" active="no"/>
-<layer number="49" name="Reference" color="7" fill="1" visible="yes" active="no"/>
-<layer number="50" name="dxf" color="7" fill="1" visible="yes" active="no"/>
-<layer number="51" name="tDocu" color="7" fill="1" visible="yes" active="no"/>
-<layer number="52" name="bDocu" color="7" fill="1" visible="yes" active="no"/>
-<layer number="53" name="tGND_GNDA" color="7" fill="9" visible="yes" active="no"/>
-<layer number="54" name="bGND_GNDA" color="1" fill="9" visible="yes" active="no"/>
-<layer number="56" name="wert" color="7" fill="1" visible="yes" active="no"/>
-<layer number="57" name="tCAD" color="7" fill="1" visible="yes" active="no"/>
+<layer number="46" name="Milling" color="3" fill="1" visible="no" active="no"/>
+<layer number="47" name="Measures" color="7" fill="1" visible="no" active="no"/>
+<layer number="48" name="Document" color="7" fill="1" visible="no" active="no"/>
+<layer number="49" name="Reference" color="7" fill="1" visible="no" active="no"/>
+<layer number="50" name="dxf" color="7" fill="1" visible="no" active="no"/>
+<layer number="51" name="tDocu" color="7" fill="1" visible="no" active="no"/>
+<layer number="52" name="bDocu" color="7" fill="1" visible="no" active="no"/>
+<layer number="53" name="tGND_GNDA" color="7" fill="9" visible="no" active="no"/>
+<layer number="54" name="bGND_GNDA" color="1" fill="9" visible="no" active="no"/>
+<layer number="56" name="wert" color="7" fill="1" visible="no" active="no"/>
+<layer number="57" name="tCAD" color="7" fill="1" visible="no" active="no"/>
 <layer number="90" name="Modules" color="5" fill="1" visible="yes" active="yes"/>
 <layer number="91" name="Nets" color="2" fill="1" visible="yes" active="yes"/>
@@
 <instance part="JP2" gate="A" x="27.94" y="137.16" rot="R90"/>
 <instance part="JP3" gate="A" x="40.64" y="104.14"/>
-<instance part="GND8" gate="1" x="15.24" y="104.14"/>
+<instance part="GND8" gate="1" x="15.24" y="109.22"/>
 <instance part="TP1" gate="G$1" x="335.28" y="246.38"/>
 <instance part="GND12" gate="1" x="256.54" y="203.2"/>
@@
 </segment>
 <segment>
-<pinref part="JP3" gate="A" pin="3"/>
-<pinref part="GND8" gate="1" pin="GND"/>
-<wire x1="15.24" y1="106.68" x2="38.1" y2="106.68" width="0.1524" layer="91"/>
-</segment>
-<segment>
 <pinref part="GND12" gate="1" pin="GND"/>
 <wire x1="254" y1="205.74" x2="256.54" y2="205.74" width="0.1524" layer="91"/>
@@
 <wire x1="63.5" y1="45.72" x2="63.5" y2="48.26" width="0.1524" layer="91"/>
 <pinref part="IC3" gate="G$1" pin="V-"/>
+</segment>
+<segment>
+<wire x1="15.24" y1="111.76" x2="38.1" y2="111.76" width="0.1524" layer="91"/>
+<pinref part="GND8" gate="1" pin="GND"/>
+<pinref part="JP3" gate="A" pin="1"/>
 </segment>
 </net>
@@
 </segment>
 <segment>
-<wire x1="17.78" y1="127" x2="17.78" y2="134.62" width="0.1524" layer="91"/>
-<label x="12.7" y="124.46" size="1.778" layer="95"/>
-<pinref part="JP2" gate="A" pin="1"/>
-</segment>
-<segment>
 <wire x1="254" y1="198.12" x2="259.08" y2="198.12" width="0.1524" layer="91"/>
 <pinref part="U$4" gate="G$1" pin="SDA"/>
+</segment>
+<segment>
+<wire x1="20.32" y1="127" x2="20.32" y2="134.62" width="0.1524" layer="91"/>
+<pinref part="JP2" gate="A" pin="2"/>
 </segment>
 </net>
@@
 </segment>
 <segment>
-<wire x1="20.32" y1="134.62" x2="20.32" y2="121.92" width="0.1524" layer="91"/>
-<label x="20.32" y="119.38" size="1.778" layer="95"/>
-<pinref part="JP2" gate="A" pin="2"/>
-</segment>
-<segment>
 <wire x1="218.44" y1="198.12" x2="228.6" y2="198.12" width="0.1524" layer="91"/>
 <pinref part="U$4" gate="G$1" pin="SCL"/>
+</segment>
+<segment>
+<wire x1="17.78" y1="134.62" x2="17.78" y2="121.92" width="0.1524" layer="91"/>
+<pinref part="JP2" gate="A" pin="1"/>
 </segment>
 </net>
@@
 </segment>
 <segment>
-<wire x1="22.86" y1="111.76" x2="38.1" y2="111.76" width="0.1524" layer="91"/>
-<label x="15.24" y="111.76" size="1.778" layer="95"/>
-<pinref part="JP3" gate="A" pin="1"/>
-</segment>
-<segment>
 <wire x1="66.04" y1="142.24" x2="83.82" y2="142.24" width="0.1524" layer="91"/>
 <label x="58.42" y="142.24" size="1.778" layer="95"/>
 <pinref part="JP4" gate="A" pin="1"/>
 </segment>
-</net>
+<segment>
+<wire x1="22.86" y1="106.68" x2="38.1" y2="106.68" width="0.1524" layer="91"/>
+<label x="22.86" y="101.6" size="1.778" layer="95"/>
+<pinref part="JP3" gate="A" pin="3"/>
+</segment>
+</net>
