File: Arduino/hardware/proposed/building blocks/AVR/AVR.brd (EAGLE design)
At the start: 36.8 x 30.9 mm, 39 parts, among them IC2 ATMEGA168-AU, Q1 32768Hz

Commit message: a few ideas for modular building blocks
Parts:
- moved PAD13 25.4 mm to (26.7, 0.00)
- moved PAD12 20.3 mm to (24.1, 0.00)
- moved PAD4 17.8 mm to (6.35, 0.00)
- moved PAD5 12.7 mm to (8.89, 0.00)
- moved PAD1 10.2 mm to (21.6, 0.00)
- moved PAD10 7.62 mm to (1.27, 0.00)
- moved PAD6 7.62 mm to (11.4, 0.00)
- moved PAD9 7.62 mm to (19.1, 0.00)
- moved PAD15 6.35 mm to (35.6, 30.9)
- moved PAD16 6.35 mm to (33.0, 30.9)
- moved PAD22 6.35 mm to (17.8, 30.9)
- moved PAD25 6.35 mm to (10.2, 30.9)
- moved PAD3 5.08 mm to (31.8, 0.00)
- moved PAD17 3.81 mm to (27.9, 30.9)
- moved PAD18 3.81 mm to (25.4, 30.9)
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Routing:
- net GND: track 3.03 -> 104.5 mm
- net N$4: track 57.2 -> 26.6 mm, vias 4 -> 1
- net TX: track 58.2 -> 31.0 mm, vias 3 -> 2
- net RX: track 59.0 -> 34.3 mm, vias 5 -> 3
- net N$5: track 29.8 -> 9.43 mm, vias 1 -> 0
- net N$2: track 29.9 -> 10.4 mm, vias 3 -> 0
- net VCC: track 80.6 -> 99.7 mm, vias 0 -> 1
- net RESET: track 54.8 -> 36.6 mm, vias 3 -> 2
- net SDA: track 49.6 -> 35.1 mm, vias 3 -> 1
- net SCL: track 47.8 -> 34.3 mm
- net D2: track 57.7 -> 49.7 mm, vias 0 -> 1
- net N$7: track 16.5 -> 9.29 mm, vias 1 -> 0
- net N$13: track 18.3 -> 24.4 mm, vias 2 -> 1
- net N$9: track 35.3 -> 40.1 mm
- net N$12: track 21.8 -> 26.2 mm, vias 2 -> 1
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- removed copper zone on layer 1, net GND
- removed copper zone on layer 16, net GND
