File: Arduino/hardware/REV15/rev15.sch (EAGLE design)
At the start: 18 parts, among them IC2 ATMEGA168-AU, Q1 32768Hz

Commit message: up to rev18 cleaned up
Changed lines of the file:
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@@
 <text x="7.62" y="10.16" size="1.778" layer="91">OF ANY KIND, either express or implied. See the Licence for the</text>
 <text x="7.62" y="7.62" size="1.778" layer="91">specific language governing permissions and limitations under the Licence.</text>
-<wire x1="93.98" y1="208.28" x2="45.72" y2="208.28" width="0.3048" layer="94"/>
 <wire x1="45.72" y1="208.28" x2="0" y2="208.28" width="0.3048" layer="94"/>
 <wire x1="157.48" y1="208.28" x2="157.48" y2="264.16" width="0.3048" layer="94"/>

Commit message: REV15-18 cleaned up, need sanity check
Other:
- note added: "Author(s) / Copyright (s): Bo Herrmannsen 2013--2016, Damon Hart-Davis 2013--2016, Mike Stirling 2013"
- note removed: "Author(s) / Copyright (s): Bo Herrmannsen 2013--2014, Damon Hart-Davis 2013--2014, Mike Stirling 2013"
- note removed: "OpenTRV Wireless TRV Controller"
Changed lines of the file:
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@@
 <text x="7.62" y="15.24" size="1.778" layer="91">software, hardware and materials distributed under this Licence</text>
 <text x="7.62" y="12.7" size="1.778" layer="91">is distributed on an "AS IS" BASIS, WITHOUT WARRANTIES OR CONDITIONS</text>
-<text x="7.62" y="2.54" size="1.778" layer="91">Author(s) / Copyright (s): Bo Herrmannsen 2013--2014, Damon Hart-Davis 2013--2014, Mike Stirling 2013</text>
-<text x="289.56" y="33.02" size="1.778" layer="91">OpenTRV Wireless TRV Controller</text>
+<text x="7.62" y="2.54" size="1.778" layer="91">Author(s) / Copyright (s): Bo Herrmannsen 2013--2016, Damon Hart-Davis 2013--2016, Mike Stirling 2013</text>
 <text x="7.62" y="10.16" size="1.778" layer="91"></text>
 <text x="7.62" y="10.16" size="1.778" layer="91">OF ANY KIND, either express or implied. See the Licence for the</text>
