File: Arduino/hardware/REV15/REV17/rev17.sch (EAGLE design)
At the start: 7 parts

Commit message: up to rev18 cleaned up
Connections:
- removed net N$20: RFM22B.GPIO0, RFM22B.RXANT
- removed net N$21: RFM22B.GPIO1, RFM22B.TXANT
Changed lines of the file:
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@@
-</segment>
-</net>
-<net name="N$20" class="0">
-<segment>
-<pinref part="RFM22B" gate="G$1" pin="RXANT"/>
-<wire x1="142.24" y1="157.48" x2="147.32" y2="157.48" width="0.1524" layer="91"/>
-<pinref part="RFM22B" gate="G$1" pin="GPIO0"/>
-<wire x1="147.32" y1="149.86" x2="142.24" y2="149.86" width="0.1524" layer="91"/>
-<wire x1="147.32" y1="157.48" x2="147.32" y2="149.86" width="0.1524" layer="91"/>
-</segment>
-</net>
-<net name="N$21" class="0">
-<segment>
-<pinref part="RFM22B" gate="G$1" pin="TXANT"/>
-<wire x1="142.24" y1="154.94" x2="149.86" y2="154.94" width="0.1524" layer="91"/>
-<pinref part="RFM22B" gate="G$1" pin="GPIO1"/>
-<wire x1="149.86" y1="147.32" x2="142.24" y2="147.32" width="0.1524" layer="91"/>
-<wire x1="149.86" y1="154.94" x2="149.86" y2="147.32" width="0.1524" layer="91"/>
 </segment>
 </net>

Commit message: REV15-18 cleaned up, need sanity check
Other:
- note added: "Author(s) / Copyright (s): Bo Herrmannsen 2013--2016, Damon Hart-Davis 2013--2016, Mike Stirling 2013"
- note removed: "Author(s) / Copyright (s): Bo Herrmannsen 2013--2014, Damon Hart-Davis 2013--2014, Mike Stirling 2013"
- note removed: "OpenTRV Wireless TRV Controller"
Changed lines of the file:
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@@
 <text x="7.62" y="15.24" size="1.778" layer="91">software, hardware and materials distributed under this Licence</text>
 <text x="7.62" y="12.7" size="1.778" layer="91">is distributed on an "AS IS" BASIS, WITHOUT WARRANTIES OR CONDITIONS</text>
-<text x="7.62" y="2.54" size="1.778" layer="91">Author(s) / Copyright (s): Bo Herrmannsen 2013--2014, Damon Hart-Davis 2013--2014, Mike Stirling 2013</text>
-<text x="289.56" y="33.02" size="1.778" layer="91">OpenTRV Wireless TRV Controller</text>
+<text x="7.62" y="2.54" size="1.778" layer="91">Author(s) / Copyright (s): Bo Herrmannsen 2013--2016, Damon Hart-Davis 2013--2016, Mike Stirling 2013</text>
 <text x="7.62" y="10.16" size="1.778" layer="91"></text>
 <text x="7.62" y="10.16" size="1.778" layer="91">OF ANY KIND, either express or implied. See the Licence for the</text>
