File: Arduino/hardware/rev11_Motordriver_eval/rev11.brd (EAGLE design)
At the start: 71 x 53 mm, 42 parts, among them IC2 ATMEGA168-AU, Q1 32768Hz, U1 DRV8850_RGY_24

Commit message: motor eval board as pr deniz request
Parts:
- removed JP4: (no value), pinhead:1X04
- removed NSLEEP: WIREPAD2,15/1,0, wirepad:2,15/1,0
Connections:
- removed net N$17: R14.2, U1.16
- removed net N$19: JP4.1, U1.8
- removed net N$21: JP4.2, U1.7
- removed net N$22: JP4.3, U1.6
- removed net N$24: JP4.4, U1.5
- removed net N$8: NSLEEP.1, U1.9
- net A1: now also R14.2, U1.16
- net D3: now also U1.5
- net D5: now also U1.7
- net D6: now also U1.6
- net D7: now also U1.8
- net IO_POWER_UP: now also U1.9
Routing:
- net IO_POWER_UP: track 29.8 -> 112.4 mm, vias 2 -> 3
- net A1: track 17.7 -> 58.2 mm, vias 1 -> 2
- net D7: track 44.6 -> 79.8 mm, vias 2 -> 3
- net D6: track 39.6 -> 73.3 mm, vias 2 -> 3
- net D3: track 22.1 -> 54.7 mm, vias 2 -> 3
- net D5: track 34.6 -> 67.0 mm, vias 2 -> 3
- net GND: track 35.8 -> 47.6 mm
- net N$17: track 7.58 -> 0.00 mm
- net N$8: track 7.44 -> 0.00 mm
- net N$24: track 6.53 -> 0.00 mm
- net N$22: track 5.57 -> 0.00 mm
- net N$19: track 5.36 -> 0.00 mm
- net N$21: track 4.73 -> 0.00 mm
- net VCC: track 218.9 -> 219.9 mm
