File: Arduino/hardware/rev11_Motordriver_eval/rev11.sch (EAGLE design)
At the start: 40 parts, among them IC2 ATMEGA168-AU, Q1 32768Hz, U1 DRV8850_RGY_24

Commit message: motor eval board as pr deniz request
Parts:
- removed JP4: (no value), pinhead:PINHD-1X4
- removed NSLEEP: WIREPAD2,15/1,0, wirepad:WIREPAD2,15/1,0
Connections:
- removed net N$17: R14.2, U1.VPROPI
- removed net N$19: JP4.1, U1.IN2L
- removed net N$21: JP4.2, U1.IN2H
- removed net N$22: JP4.3, U1.IN1L
- removed net N$24: JP4.4, U1.IN1H
- removed net N$8: NSLEEP.P, U1.NSLEEP
- net A1: now also R14.2, U1.VPROPI
- net D3: now also U1.IN1H
- net D5: now also U1.IN2H
- net D6: now also U1.IN1L
- net D7: now also U1.IN2L
- net IO_POWER_UP: now also U1.NSLEEP
Changed lines of the file:
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@@
 <part name="C5" library="resistor" deviceset="C-EU" device="C0603" value="10uF"/>
 <part name="GND9" library="SparkFun-Aesthetics" deviceset="GND" device=""/>
-<part name="NSLEEP" library="wirepad" deviceset="WIREPAD" device="2,15/1,0"/>
 <part name="LDOEN" library="wirepad" deviceset="WIREPAD" device="2,15/1,0"/>
-<part name="JP4" library="pinhead" deviceset="PINHD-1X4" device=""/>
 </parts>
 <sheets>
@@
 <instance part="C5" gate="G$1" x="30.48" y="91.44" rot="R180"/>
 <instance part="GND9" gate="1" x="35.56" y="86.36"/>
-<instance part="NSLEEP" gate="G$1" x="48.26" y="137.16"/>
-<instance part="LDOEN" gate="G$1" x="35.56" y="139.7"/>
-<instance part="JP4" gate="A" x="43.18" y="127" rot="R180"/>
+<instance part="LDOEN" gate="G$1" x="35.56" y="139.7" smashed="yes">
+<attribute name="NAME" x="26.797" y="139.0142" size="1.778" layer="95"/>
+</instance>
 </instances>
 <busses>
@@
 <pinref part="JP1" gate="G$1" pin="8"/>
 </segment>
+<segment>
+<wire x1="50.8" y1="124.46" x2="48.26" y2="124.46" width="0.1524" layer="91"/>
+<label x="45.72" y="124.46" size="1.778" layer="95"/>
+<pinref part="U1" gate="A" pin="IN1L"/>
+</segment>
 </net>
 <net name="SPI_SCK" class="0">
@@
 <pinref part="JP1" gate="G$1" pin="7"/>
 </segment>
+<segment>
+<wire x1="50.8" y1="127" x2="48.26" y2="127" width="0.1524" layer="91"/>
+<label x="45.72" y="127" size="1.778" layer="95"/>
+<pinref part="U1" gate="A" pin="IN2H"/>
+</segment>
 </net>
 <net name="D7" class="0">
@@
 <pinref part="JP1" gate="G$1" pin="9"/>
 </segment>
+<segment>
+<wire x1="50.8" y1="121.92" x2="48.26" y2="121.92" width="0.1524" layer="91"/>
+<label x="45.72" y="121.92" size="1.778" layer="95"/>
+<pinref part="U1" gate="A" pin="IN2L"/>
+</segment>
 </net>
 <net name="D2" class="0">
@@
 <pinref part="JP1" gate="G$1" pin="1"/>
 </segment>
+<segment>
+<pinref part="U1" gate="A" pin="VPROPI"/>
+<wire x1="50.8" y1="134.62" x2="40.64" y2="134.62" width="0.1524" layer="91"/>
+<wire x1="40.64" y1="134.62" x2="40.64" y2="121.92" width="0.1524" layer="91"/>
+<pinref part="R14" gate="G$1" pin="2"/>
+<wire x1="40.64" y1="121.92" x2="35.56" y2="121.92" width="0.1524" layer="91"/>
+<label x="38.1" y="127" size="1.778" layer="95"/>
+</segment>
 </net>
 <net name="D3" class="0">
@@
 <label x="251.46" y="88.9" size="1.778" layer="95"/>
 <pinref part="JP1" gate="G$1" pin="6"/>
+</segment>
+<segment>
+<wire x1="50.8" y1="129.54" x2="48.26" y2="129.54" width="0.1524" layer="91"/>
+<label x="45.72" y="129.54" size="1.778" layer="95"/>
+<pinref part="U1" gate="A" pin="IN1H"/>
 </segment>
 </net>
@@
 <label x="251.46" y="73.66" size="1.778" layer="95"/>
 <pinref part="IC2" gate="1" pin="DIGITAL_8"/>
+</segment>
+<segment>
+<pinref part="U1" gate="A" pin="NSLEEP"/>
+<wire x1="48.26" y1="137.16" x2="50.8" y2="137.16" width="0.1524" layer="91"/>
+<label x="35.56" y="137.16" size="1.778" layer="95"/>
 </segment>
 </net>
@@
 </segment>
 </net>
-<net name="N$17" class="0">
-<segment>
-<pinref part="U1" gate="A" pin="VPROPI"/>
-<wire x1="50.8" y1="134.62" x2="40.64" y2="134.62" width="0.1524" layer="91"/>
-<wire x1="40.64" y1="134.62" x2="40.64" y2="121.92" width="0.1524" layer="91"/>
-<pinref part="R14" gate="G$1" pin="2"/>
-<wire x1="40.64" y1="121.92" x2="35.56" y2="121.92" width="0.1524" layer="91"/>
-</segment>
-</net>
 <net name="N$20" class="0">
 <segment>
@@
 </segment>
 </net>
-<net name="N$8" class="0">
-<segment>
-<pinref part="U1" gate="A" pin="NSLEEP"/>
-<pinref part="NSLEEP" gate="G$1" pin="P"/>
-</segment>
-</net>
 <net name="N$16" class="0">
 <segment>
@@
 </segment>
 </net>
-<net name="N$19" class="0">
-<segment>
-<pinref part="U1" gate="A" pin="IN2L"/>
-<pinref part="JP4" gate="A" pin="1"/>
-<wire x1="45.72" y1="121.92" x2="50.8" y2="121.92" width="0.1524" layer="91"/>
-</segment>
-</net>
-<net name="N$24" class="0">
-<segment>
-<pinref part="U1" gate="A" pin="IN1H"/>
-<pinref part="JP4" gate="A" pin="4"/>
-<wire x1="45.72" y1="129.54" x2="50.8" y2="129.54" width="0.1524" layer="91"/>
-</segment>
-</net>
-<net name="N$21" class="0">
-<segment>
-<pinref part="U1" gate="A" pin="IN2H"/>
-<wire x1="50.8" y1="127" x2="48.26" y2="127" width="0.1524" layer="91"/>
-<wire x1="48.26" y1="127" x2="48.26" y2="124.46" width="0.1524" layer="91"/>
-<pinref part="JP4" gate="A" pin="2"/>
-<wire x1="48.26" y1="124.46" x2="45.72" y2="124.46" width="0.1524" layer="91"/>
-</segment>
-</net>
-<net name="N$22" class="0">
-<segment>
-<pinref part="JP4" gate="A" pin="3"/>
-<wire x1="45.72" y1="127" x2="46.736" y2="127" width="0.1524" layer="91"/>
-<wire x1="46.736" y1="127" x2="46.736" y2="125.73" width="0.1524" layer="91"/>
-<pinref part="U1" gate="A" pin="IN1L"/>
-<wire x1="46.736" y1="125.73" x2="50.8" y2="125.73" width="0.1524" layer="91"/>
-<wire x1="50.8" y1="125.73" x2="50.8" y2="124.46" width="0.1524" layer="91"/>
-</segment>
-</net>
